File: kiCad_project/sdcb_electronic_scheme.kicad_pcb (KiCad board)
At the start: 2 copper layers, 144.8 x 99.1 mm, 82 parts, among them CON1 SD_Card, J1 POWER_12V, J10 B_RIGHT_T, J11 DB9, J12 RELAY_CONTROL, J13 HEADER_5, J2 Arduino_Nano_Header, J3 REAL_TIME_CLOCK, J4 LEFT_TURN_GYRO, J5 RIGHT_TURN_GYRO, J6 POWER_MOTOR, J7 MOTOR, J8 DB15, J9 B_LEFT_T, Q1 BC817-40, Q2 BC817-40, Q3 BC817-40, U2 74HC595, U3 74HC595, U4 74HC595, U5 LTV-817, U6 LTV-817, U7 LTV-817

Commit message: Varžtai IN
Parts:
- added C3: 2200uF >6.3V, Capacitors_Elko_ThroughHole:Elko_vert_25x14mm_RM5_CopperClear, F.Cu at (110.7, 64.0)
- added J14: HEADER_1, Mounting_Holes:MountingHole_3-7mm, F.Cu at (145.3, 82.8)
- added J15: HEADER_1, Mounting_Holes:MountingHole_3-7mm, F.Cu at (193.0, 97.0)
- Q2: footprint Housings_TO-92:TO-92_Molded_Wide_Oval -> Housings_TO-92:TO-92_Inline_Wide
- moved R15 11.3 mm to (104.9, 55.6), turned to 90 degrees
- moved R13 11.3 mm to (118.9, 59.9), turned to 90 degrees
- moved R18 7.03 mm to (126.5, 70.1)
- moved U6 5.45 mm to (109.0, 57.7), turned to 90 degrees
- moved D35 3.54 mm to (123.4, 63.5)
- moved J5 2.67 mm to (127.0, 64.0)
- moved D11 2.30 mm to (130.6, 136.7)
- moved D9 2.30 mm to (133.1, 136.7)
- moved Q2 1.93 mm to (115.3, 51.3), turned to 0 degrees
Connections:
- J4 pad 4: Net-(J4-Pad4) -> VCC
- J5 pad 4: Net-(J4-Pad4) -> VCC
- R18 pad 1: Net-(J4-Pad4) -> VCC
Routing:
- net VCC: track 261.4 -> 365.2 mm
- net Net-(D35-Pad2): track 18.7 -> 8.78 mm
- net Net-(J4-Pad4): track 8.13 -> 0.00 mm
- net Net-(J2-Pad7): track 53.7 -> 45.6 mm
- net Net-(R13-Pad1): track 3.00 -> 10.4 mm
- net Net-(Q2-Pad1): track 11.7 -> 4.34 mm
- net GND: track 236.4 -> 240.5 mm
- net Net-(J7-Pad2): track 56.4 -> 59.6 mm
- net Net-(D11-Pad1): track 3.21 -> 5.40 mm
- net Net-(R15-Pad2): track 6.22 -> 4.27 mm
- net Net-(D36-Pad2): track 15.2 -> 14.2 mm
- net Net-(Current1-Pad1): track 50.7 -> 49.7 mm
- net Net-(D9-Pad1): track 4.21 -> 3.51 mm
Other:
- board text added: "DO214AC printo ir pačių diodų. Pakeisti footprintą DB9 DB15 nusipirkti."
